File: Hardware/AC-CTRL-BRD.sch (EAGLE design)
At the start: 17 parts, among them IC1 ULN2803AGP, IC2 ULN2803AGP, IC3 MCP23017, K1 JW1A, K2 JW1A, K3 JW1A, K4 JW1A, K5 JW1A, X1 SMKDSP_1,5/12, X2 SMKDSP_1,5/12

Commit message: continued board work
Connections:
- net N$23: now also X1-11.KL; no longer X1-1.KL
- net N$24: now also X1-12.KL; no longer X1-2.KL
- net N$25: now also X1-9.KL; no longer X1-3.KL
- net N$26: now also X1-10.KL; no longer X1-4.KL
- net N$27: now also X1-7.KL; no longer X1-5.KL
- net N$28: now also X1-8.KL; no longer X1-6.KL
- net N$29: now also X1-5.KL; no longer X1-7.KL
- net N$30: now also X1-6.KL; no longer X1-8.KL
- net N$31: now also K51.P, X1-4.KL; no longer K51.S, X1-9.KL
- net N$32: now also K51.S, X1-3.KL; no longer K51.P, X1-10.KL
- net N$33: now also X2-12.KL; no longer X2-2.KL
- net N$34: now also X2-10.KL; no longer X2-4.KL
- net N$35: now also X2-8.KL; no longer X2-6.KL
- net N$36: now also X2-6.KL; no longer X2-8.KL
- net N$37: now also X2-4.KL; no longer X2-10.KL
- net N$38: now also X2-2.KL; no longer X2-12.KL
- net SCL: now also JP1.6; no longer JP1.5
- net SDA: now also JP1.5; no longer JP1.6
Other:
- moved on the sheet: X1-1, X1-10, X1-11, X1-12, X1-2, X1-3, X1-4, X1-5, X1-6, X1-7, X1-8, X1-9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
